File: 5Vin_3.3Vout_Regulator.kicad_sch (KiCad schematic)
At the start: 4 parts, among them J1 PinSocket_1x04_P2.54mm_Vertic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, U1 AP2112K-3.3

Commit message: Change connector name from socket to header. Some minor traces changes.
Parts:
- J1: value PinSocket_1x04_P2.54mm_Vertical_SMD_Pin1Left -> PinHeader_1x04_P2.54mm_Vertical_SMD_Pin1Left; footprint Library:PinSocket_1x04_P2.54mm_Vertical_SMD_Pin1Left -> PnP_Library:PinSocket_1x04_P2.54mm_Vertical_SMD_Pin1Left
Changed lines of the file:
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@@
 (kicad_sch
-	(version 20231120)
+	(version 20250114)
 	(generator "eeschema")
-	(generator_version "8.0")
+	(generator_version "9.0")
 	(paper "A5")
 	(title_block
@@
 			)
 		)
-		(property "Value" "PinSocket_1x04_P2.54mm_Vertical_SMD_Pin1Left"
+		(property "Value" "PinHeader_1x04_P2.54mm_Vertical_SMD_Pin1Left"
 			(at 30.48 34.29 0)
 			(effects
@@
 			)
 		)
-		(property "Footprint" "Library:PinSocket_1x04_P2.54mm_Vertical_SMD_Pin1Left"
+		(property "Footprint" "PnP_Library:PinSocket_1x04_P2.54mm_Vertical_SMD_Pin1Left"
 			(at 36.83 33.02 0)
 			(effects
@@
 		)
 		(instances
-			(project ""
+			(project "5Vin_3.3Vout_Regulator"
 				(path "/1a1c72da-99f5-4976-b608-38ee505f2b67"
 					(reference "C2")
@@
 		)
 		(instances
-			(project ""
+			(project "5Vin_3.3Vout_Regulator"
 				(path "/1a1c72da-99f5-4976-b608-38ee505f2b67"
 					(reference "U1")
@@
 		)
 		(instances
-			(project ""
+			(project "5Vin_3.3Vout_Regulator"
 				(path "/1a1c72da-99f5-4976-b608-38ee505f2b67"
 					(reference "#PWR01")
@@
 		)
 		(instances
-			(project ""
+			(project "5Vin_3.3Vout_Regulator"
 				(path "/1a1c72da-99f5-4976-b608-38ee505f2b67"
 					(reference "C1")
@@
 		)
 	)
+	(embedded_fonts no)
 )
